File: pcb/_saved_padma1Ver2.sch (KiCad schematic (older format))
At the start: 15 parts, among them SW1 SPST, U1 NodeMCU_Amica_R2

Commit message: added WebApp files by Prof A Mohan
Parts:
- SW1: footprint (none) -> Buttons_Switches_SMD:SW_SPST_EVPBF
- renumbered 2n1 to 2n3906, U1 to u**1
Changed lines of the file:
@@
 F 0 "R3" V 5680 4650 50  0000 C CNN
 F 1 "R" V 5600 4650 50  0000 C CNN
-F 2 "" V 5530 4650 50  0000 C CNN
+F 2 "" V 5530 4650 50  0001 C CNN
 F 3 "" H 5600 4650 50  0000 C CNN
 	1    5600 4650
@@
 F 0 "10k1" V 5530 3100 50  0000 C CNN
 F 1 "R" V 5450 3100 50  0000 C CNN
-F 2 "" V 5380 3100 50  0000 C CNN
+F 2 "" V 5380 3100 50  0001 C CNN
 F 3 "" H 5450 3100 50  0000 C CNN
 	1    5450 3100
@@
 F 0 "D2" H 3650 3000 50  0000 C CNN
 F 1 "D" H 3650 2800 50  0000 C CNN
-F 2 "" H 3650 2900 50  0000 C CNN
+F 2 "" H 3650 2900 50  0001 C CNN
 F 3 "" H 3650 2900 50  0000 C CNN
 	1    3650 2900
@@
 $EndComp
 $Comp
-L Q_PNP_BCE 2n1
+L Q_PNP_BCE 2n3906
 U 1 1 582C37C4
 P 5950 3100
-F 0 "2n1" H 6250 3150 50  0000 C CNN
+F 0 "2n3906" H 6250 3150 50  0000 C CNN
 F 1 "Q_PNP_BCE" H 6550 3050 50  0001 R CNN
-F 2 "" H 6150 3200 50  0000 C CNN
+F 2 "" H 6150 3200 50  0001 C CNN
 F 3 "" H 5950 3100 50  0000 C CNN
 	1    5950 3100
@@
 F 0 "SW1" H 6100 4450 50  0000 C CNN
 F 1 "SPST" H 6100 4250 50  0000 C CNN
-F 2 "" H 6100 4350 50  0000 C CNN
+F 2 "Buttons_Switches_SMD:SW_SPST_EVPBF" H 6100 4350 50  0001 C CNN
 F 3 "" H 6100 4350 50  0000 C CNN
 	1    6100 4350
@@
 F 0 "D1" H 3650 2700 50  0000 C CNN
 F 1 "D" H 3650 2500 50  0000 C CNN
-F 2 "" H 3650 2600 50  0000 C CNN
+F 2 "" H 3650 2600 50  0001 C CNN
 F 3 "" H 3650 2600 50  0000 C CNN
 	1    3650 2600
@@
 F 0 "LDR1" H 4600 2300 50  0000 C CNN
 F 1 "CONN_01X04" V 4700 2050 50  0001 C CNN
-F 2 "" H 4600 2050 50  0000 C CNN
+F 2 "" H 4600 2050 50  0001 C CNN
 F 3 "" H 4600 2050 50  0000 C CNN
 	1    4600 2050
@@
 F 0 "MOIS1" H 4600 1750 50  0000 C CNN
 F 1 "CONN_01X04" V 4700 1500 50  0001 C CNN
-F 2 "" H 4600 1500 50  0000 C CNN
+F 2 "" H 4600 1500 50  0001 C CNN
 F 3 "" H 4600 1500 50  0000 C CNN
 	1    4600 1500
@@
 F 0 "DTH1" H 5850 2300 50  0000 C CNN
 F 1 "CONN_01X04" V 5950 2050 50  0001 C CNN
-F 2 "" H 5850 2050 50  0000 C CNN
+F 2 "" H 5850 2050 50  0001 C CNN
 F 3 "" H 5850 2050 50  0000 C CNN
 	1    5850 2050
@@
 F 0 "Grovr1" H 6650 3200 50  0001 C CNN
 F 1 "RLY" H 6750 2950 50  0000 C CNN
-F 2 "" H 6650 2950 50  0000 C CNN
+F 2 "" H 6650 2950 50  0001 C CNN
 F 3 "" H 6650 2950 50  0000 C CNN
 	1    6650 2950
@@
 F 0 "D3" H 6050 4050 50  0000 C CNN
 F 1 "LED_RCBG" H 6050 3350 50  0000 C CNN
-F 2 "" H 6050 3650 50  0000 C CNN
+F 2 "" H 6050 3650 50  0001 C CNN
 F 3 "" H 6050 3650 50  0000 C CNN
 	1    6050 3700
@@
 F 0 "R4" V 5730 3350 50  0000 C CNN
 F 1 "R" V 5650 3350 50  0000 C CNN
-F 2 "" V 5580 3350 50  0000 C CNN
+F 2 "" V 5580 3350 50  0001 C CNN
 F 3 "" H 5650 3350 50  0000 C CNN
 	1    5650 3350
@@
 F 0 "R1" V 5580 3550 50  0000 C CNN
 F 1 "R" V 5500 3550 50  0000 C CNN
-F 2 "" V 5430 3550 50  0000 C CNN
+F 2 "" V 5430 3550 50  0001 C CNN
 F 3 "" H 5500 3550 50  0000 C CNN
 	1    5500 3550
@@
 F 0 "R2" V 5580 3900 50  0000 C CNN
 F 1 "R" V 5500 3900 50  0000 C CNN
-F 2 "" V 5430 3900 50  0000 C CNN
+F 2 "" V 5430 3900 50  0001 C CNN
 F 3 "" H 5500 3900 50  0000 C CNN
 	1    5500 3900
@@
 NoConn ~ 4200 3900
 $Comp
-L NodeMCU_Amica_R2 U1
+L NodeMCU_Amica_R2 u**1
 U 1 1 582C3605
 P 4650 3500
-F 0 "U1" H 4650 4300 50  0000 C CNN
+F 0 "u**1" H 4650 4300 50  0000 C CNN
 F 1 "NodeMCU_Amica_R2" H 4650 2650 50  0000 C CNN
-F 2 "" H 4900 3500 50  0000 C CNN
+F 2 "" H 4900 3500 50  0001 C CNN
 F 3 "" H 4900 3500 50  0000 C CNN
 	1    4650 3500
