File: pcb/padma1Ver2.sch (KiCad schematic (older format))
At the start: 15 parts, among them SW1 SPST

Commit message: added basic PCB
Parts:
- 10k1, R1, R2, R3, R4: footprint (none) -> Resistors_ThroughHole:Resistor_Horizontal_RM10mm
- 2n3906: footprint (none) -> TO_SOT_Packages_THT:TO-92_Molded_Wide
- D1, D2: footprint (none) -> Diodes_ThroughHole:Diode_DO-35_SOD27_Horizontal_RM10
- D3: footprint (none) -> LEDs:LED-RGB-5MM_Common_Cathode
- DTH1, Grovr1, LDR1, MOIS1: footprint (none) -> Pin_Headers:Pin_Header_Straight_1x04
- nodemcu1: footprint (none) -> nodemcu:NodeMCU_Amica_R2
Connections:
- net signal: now reaches DTH1.1 (P1), nodemcu1.28 (D2)
- net signal: now also D1.2 (A), D2.2 (A), LDR1.1 (P1), MOIS1.1 (P1)
- net power: now reaches MOIS1.3 (P3), nodemcu1.29 (D1)
- net power: now also LDR1.3 (P3), nodemcu1.30 (D0)
Changed lines of the file:
@@
 LIBS:nodemcu
 LIBS:w_relay
-LIBS:padma1Ver2-cache
 EELAYER 25 0
 EELAYER END
@@
 F 0 "R3" V 5680 4650 50  0000 C CNN
 F 1 "R" V 5600 4650 50  0000 C CNN
-F 2 "" V 5530 4650 50  0001 C CNN
+F 2 "Resistors_ThroughHole:Resistor_Horizontal_RM10mm" V 5530 4650 50  0001 C CNN
 F 3 "" H 5600 4650 50  0000 C CNN
 	1    5600 4650
@@
 F 0 "10k1" V 5530 3100 50  0000 C CNN
 F 1 "R" V 5450 3100 50  0000 C CNN
-F 2 "" V 5380 3100 50  0001 C CNN
+F 2 "Resistors_ThroughHole:Resistor_Horizontal_RM10mm" V 5380 3100 50  0001 C CNN
 F 3 "" H 5450 3100 50  0000 C CNN
 	1    5450 3100
@@
 F 0 "D2" H 3650 3000 50  0000 C CNN
 F 1 "D" H 3650 2800 50  0000 C CNN
-F 2 "" H 3650 2900 50  0001 C CNN
+F 2 "Diodes_ThroughHole:Diode_DO-35_SOD27_Horizontal_RM10" H 3650 2900 50  0001 C CNN
 F 3 "" H 3650 2900 50  0000 C CNN
 	1    3650 2900
@@
 F 0 "2n3906" H 6250 3150 50  0000 C CNN
 F 1 "Q_PNP_BCE" H 6550 3050 50  0001 R CNN
-F 2 "" H 6150 3200 50  0001 C CNN
+F 2 "TO_SOT_Packages_THT:TO-92_Molded_Wide" H 6150 3200 50  0001 C CNN
 F 3 "" H 5950 3100 50  0000 C CNN
 	1    5950 3100
@@
 F 0 "D1" H 3650 2700 50  0000 C CNN
 F 1 "D" H 3650 2500 50  0000 C CNN
-F 2 "" H 3650 2600 50  0001 C CNN
+F 2 "Diodes_ThroughHole:Diode_DO-35_SOD27_Horizontal_RM10" H 3650 2600 50  0001 C CNN
 F 3 "" H 3650 2600 50  0000 C CNN
 	1    3650 2600
@@
 F 0 "LDR1" H 4600 2300 50  0000 C CNN
 F 1 "CONN_01X04" V 4700 2050 50  0001 C CNN
-F 2 "" H 4600 2050 50  0001 C CNN
+F 2 "Pin_Headers:Pin_Header_Straight_1x04" H 4600 2050 50  0001 C CNN
 F 3 "" H 4600 2050 50  0000 C CNN
 	1    4600 2050
@@
 F 0 "MOIS1" H 4600 1750 50  0000 C CNN
 F 1 "CONN_01X04" V 4700 1500 50  0001 C CNN
-F 2 "" H 4600 1500 50  0001 C CNN
+F 2 "Pin_Headers:Pin_Header_Straight_1x04" H 4600 1500 50  0001 C CNN
 F 3 "" H 4600 1500 50  0000 C CNN
 	1    4600 1500
@@
 F 0 "DTH1" H 5850 2300 50  0000 C CNN
 F 1 "CONN_01X04" V 5950 2050 50  0001 C CNN
-F 2 "" H 5850 2050 50  0001 C CNN
+F 2 "Pin_Headers:Pin_Header_Straight_1x04" H 5850 2050 50  0001 C CNN
 F 3 "" H 5850 2050 50  0000 C CNN
 	1    5850 2050
@@
 F 0 "Grovr1" H 6650 3200 50  0001 C CNN
 F 1 "RLY" H 6750 2950 50  0000 C CNN
-F 2 "" H 6650 2950 50  0001 C CNN
+F 2 "Pin_Headers:Pin_Header_Straight_1x04" H 6650 2950 50  0001 C CNN
 F 3 "" H 6650 2950 50  0000 C CNN
 	1    6650 2950
@@
 NoConn ~ 4550 1700
 $Comp
-L Earth #PWR2
+L Earth #PWR01
 U 1 1 582C4AC2
 P 4750 2250
-F 0 "#PWR2" H 4750 2000 50  0001 C CNN
+F 0 "#PWR01" H 4750 2000 50  0001 C CNN
 F 1 "Earth" H 4750 2100 50  0001 C CNN
 F 2 "" H 4750 2250 50  0000 C CNN
@@
 $EndComp
 $Comp
-L +3.3V #PWR8
+L +3.3V #PWR02
 U 1 1 582C5C13
 P 6050 2900
-F 0 "#PWR8" H 6050 2750 50  0001 C CNN
+F 0 "#PWR02" H 6050 2750 50  0001 C CNN
 F 1 "+3.3V" H 6050 3040 50  0000 C CNN
 F 2 "" H 6050 2900 50  0000 C CNN
@@
 $EndComp
 $Comp
-L Earth #PWR1
+L Earth #PWR03
 U 1 1 582C693C
 P 4750 1700
-F 0 "#PWR1" H 4750 1450 50  0001 C CNN
+F 0 "#PWR03" H 4750 1450 50  0001 C CNN
 F 1 "Earth" H 4750 1550 50  0001 C CNN
 F 2 "" H 4750 1700 50  0000 C CNN
@@
 NoConn ~ 5800 2250
 $Comp
-L +3.3V #PWR6
+L +3.3V #PWR04
 U 1 1 582C7499
 P 5900 2400
-F 0 "#PWR6" H 5900 2250 50  0001 C CNN
+F 0 "#PWR04" H 5900 2250 50  0001 C CNN
 F 1 "+3.3V" H 5900 2540 50  0000 C CNN
 F 2 "" H 5900 2400 50  0000 C CNN
@@
 $EndComp
 $Comp
-L Earth #PWR7
+L Earth #PWR05
 U 1 1 582C7550
 P 6000 2300
-F 0 "#PWR7" H 6000 2050 50  0001 C CNN
+F 0 "#PWR05" H 6000 2050 50  0001 C CNN
 F 1 "Earth" H 6000 2150 50  0001 C CNN
 F 2 "" H 6000 2300 50  0000 C CNN
@@
 NoConn ~ 6600 3150
 $Comp
-L +3.3V #PWR11
+L +3.3V #PWR06
 U 1 1 582C78ED
 P 6700 3350
-F 0 "#PWR11" H 6700 3200 50  0001 C CNN
+F 0 "#PWR06" H 6700 3200 50  0001 C CNN
 F 1 "+3.3V" H 6700 3490 50  0000 C CNN
 F 2 "" H 6700 3350 50  0000 C CNN
@@
 $EndComp
 $Comp
-L Earth #PWR12
+L Earth #PWR07
 U 1 1 582C79CF
 P 6800 3250
-F 0 "#PWR12" H 6800 3000 50  0001 C CNN
+F 0 "#PWR07" H 6800 3000 50  0001 C CNN
 F 1 "Earth" H 6800 3100 50  0001 C CNN
 F 2 "" H 6800 3250 50  0000 C CNN
@@
 F 0 "D3" H 6050 4050 50  0000 C CNN
 F 1 "LED_RCBG" H 6050 3350 50  0000 C CNN
-F 2 "" H 6050 3650 50  0001 C CNN
+F 2 "LEDs:LED-RGB-5MM_Common_Cathode" H 6050 3650 50  0001 C CNN
 F 3 "" H 6050 3650 50  0000 C CNN
 	1    6050 3700
@@
 F 0 "R4" V 5730 3350 50  0000 C CNN
 F 1 "R" V 5650 3350 50  0000 C CNN
-F 2 "" V 5580 3350 50  0001 C CNN
+F 2 "Resistors_ThroughHole:Resistor_Horizontal_RM10mm" V 5580 3350 50  0001 C CNN
 F 3 "" H 5650 3350 50  0000 C CNN
 	1    5650 3350
@@
 F 0 "R1" V 5580 3550 50  0000 C CNN
 F 1 "R" V 5500 3550 50  0000 C CNN
-F 2 "" V 5430 3550 50  0001 C CNN
+F 2 "Resistors_ThroughHole:Resistor_Horizontal_RM10mm" V 5430 3550 50  0001 C CNN
 F 3 "" H 5500 3550 50  0000 C CNN
 	1    5500 3550
@@
 F 0 "R2" V 5580 3900 50  0000 C CNN
 F 1 "R" V 5500 3900 50  0000 C CNN
-F 2 "" V 5430 3900 50  0001 C CNN
+F 2 "Resistors_ThroughHole:Resistor_Horizontal_RM10mm" V 5430 3900 50  0001 C CNN
 F 3 "" H 5500 3900 50  0000 C CNN
 	1    5500 3900
@@
 $EndComp
 $Comp
-L Earth #PWR9
+L Earth #PWR08
 U 1 1 582C8C6A
 P 6350 3700
-F 0 "#PWR9" H 6350 3450 50  0001 C CNN
+F 0 "#PWR08" H 6350 3450 50  0001 C CNN
 F 1 "Earth" H 6350 3550 50  0001 C CNN
 F 2 "" H 6350 3700 50  0000 C CNN
@@
 $EndComp
 $Comp
-L Earth #PWR5
+L Earth #PWR09
 U 1 1 582C92CF
 P 5600 5000
-F 0 "#PWR5" H 5600 4750 50  0001 C CNN
+F 0 "#PWR09" H 5600 4750 50  0001 C CNN
 F 1 "Earth" H 5600 4850 50  0001 C CNN
 F 2 "" H 5600 5000 50  0000 C CNN
@@
 $EndComp
 $Comp
-L +3.3V #PWR10
+L +3.3V #PWR010
 U 1 1 582C937E
 P 6600 4350
-F 0 "#PWR10" H 6600 4200 50  0001 C CNN
+F 0 "#PWR010" H 6600 4200 50  0001 C CNN
 F 1 "+3.3V" H 6600 4490 50  0000 C CNN
 F 2 "" H 6600 4350 50  0000 C CNN
@@
 $EndComp
 $Comp
-L PWR_FLAG #FLG1
+L PWR_FLAG #FLG011
 U 1 1 582CAB1D
 P 6400 2200
-F 0 "#FLG1" H 6400 2295 50  0001 C CNN
+F 0 "#FLG011" H 6400 2295 50  0001 C CNN
 F 1 "PWR_FLAG" H 6400 2380 50  0000 C CNN
 F 2 "" H 6400 2200 50  0000 C CNN
@@
 $EndComp
 $Comp
-L PWR_FLAG #FLG2
+L PWR_FLAG #FLG012
 U 1 1 582CAB85
 P 6950 4400
-F 0 "#FLG2" H 6950 4495 50  0001 C CNN
+F 0 "#FLG012" H 6950 4495 50  0001 C CNN
 F 1 "PWR_FLAG" H 6950 4580 50  0000 C CNN
 F 2 "" H 6950 4400 50  0000 C CNN
@@
 F 0 "nodemcu1" H 4650 4300 50  0000 C CNN
 F 1 "nodemcu" H 4650 2650 50  0000 C CNN
-F 2 "" H 4900 3500 50  0001 C CNN
+F 2 "nodemcu:NodeMCU_Amica_R2" H 4900 3500 50  0001 C CNN
 F 3 "" H 4900 3500 50  0000 C CNN
 	1    4650 3500
@@
 $EndComp
 $Comp
-L +3.3V #PWR4
+L +3.3V #PWR013
 U 1 1 582CBB12
 P 5100 4200
-F 0 "#PWR4" H 5100 4050 50  0001 C CNN
+F 0 "#PWR013" H 5100 4050 50  0001 C CNN
 F 1 "+3.3V" H 5100 4340 50  0000 C CNN
 F 2 "" H 5100 4200 50  0000 C CNN
@@
 $EndComp
 $Comp
-L Earth #PWR3
+L Earth #PWR014
 U 1 1 582CBC4D
 P 5100 4100
-F 0 "#PWR3" H 5100 3850 50  0001 C CNN
+F 0 "#PWR014" H 5100 3850 50  0001 C CNN
 F 1 "Earth" H 5100 3950 50  0001 C CNN
 F 2 "" H 5100 4100 50  0000 C CNN
@@
 NoConn ~ 5100 3300
 NoConn ~ 4200 4000
+Text Label 3950 1800 0    60   ~ 0
+signal
+Text Label 4900 1850 0    60   ~ 0
+power
+Text Label 3850 2350 0    60   ~ 0
+signal
+Text Label 4950 2500 0    60   ~ 0
+power
+Text Label 5400 3000 0    60   ~ 0
+signal
 $EndSCHEMATC
